Commit message: Finished part 1 of checkpoint 1

File: my_rb1_description/urdf/my_rb1_robot.urdf (robot description, URDF)
Before this commit: robot rb1_robot, 4 links, 3 joints
Links:
- added link back_caster; collision sphere radius=0.025; visual sphere radius=0.025
- added link front_caster; collision sphere radius=0.025; visual sphere radius=0.025
- added link front_laser; collision cylinder length=0.01 radius=0.008; visual cylinder length=0.01 radius=0.008
- link left_wheel: geometry collision cylinder length=.04 radius=.025; visual cylinder length=.04 radius=.025
- link right_wheel: geometry collision cylinder length=.04 radius=.025; visual cylinder length=.04 radius=.025
Joints:
- added joint base_link_back_caster_joint: type fixed, parent base_link, child back_caster, origin xyz=0.1 0 -0.15 rpy=0 0 0
- added joint base_link_front_caster_joint: type fixed, parent base_link, child front_caster, origin xyz=-0.1 0 -0.15 rpy=0 0 0
- added joint base_link_front_laser_joint: type fixed, parent base_link, child front_laser, origin xyz=0.25 0 0.08 rpy=0 0 0
- joint base_link_left_wheel_joint: origin xyz=0 -0.2 -.15 rpy=0 0 0 -> xyz=0 0.2 -.15 rpy=0 0 0
- joint base_link_right_wheel_joint: origin xyz=0 0.2 -.15 rpy=0 0 0 -> xyz=0 -0.2 -.15 rpy=0 0 0
